Commit message: added ros control

File: src/bot_description/urdf/bot.xacro (robot description, xacro)
@@ -6,7 +6,7 @@
 <link name="base_link">
   <inertial>
-    <origin rpy="0 0 0" xyz="1.313409255906936e-15 0.0 0.024960012166825512"/>
-    <mass value="0.6679552358753357"/>
-    <inertia ixx="0.001215" ixy="-0.0" ixz="0.0" iyy="0.001219" iyz="-0.0" izz="0.002333"/>
+    <origin rpy="0 0 0" xyz="-0.0009636587923201293 1.0904768733166021e-17 0.021032044779261124"/>
+    <mass value="0.11050949445484062"/>
+    <inertia ixx="9e-05" ixy="-0.0" ixz="-1e-06" iyy="9.3e-05" iyz="0.0" izz="0.00018"/>
   </inertial>
   <visual>
@@ -24,12 +24,45 @@
   </collision>
 </link>
+<link name="wheel_1_1">
+  <inertial>
+    <origin rpy="0 0 0" xyz="3.469446951953614e-18 -0.009000000000000001 1.0408340855860843e-17"/>
+    <mass value="0.0243098481570003"/>
+    <inertia ixx="3e-06" ixy="0.0" ixz="0.0" iyy="6e-06" iyz="-0.0" izz="3e-06"/>
+  </inertial>
+  <visual>
+    <geometry>
+      <cylinder length="0.018" radius="0.0215"/>
+    </geometry>
+    <material name="black">
+      <color rgba="0 0 0 1"/>
+    </material>
+  </visual>
+  <collision>
+    <geometry>
+      <cylinder length="0.018" radius="0.0215"/>
+    </geometry>
+  </collision>
+</link>
 <link name="wheel_2_1">
   <inertial>
-    <origin rpy="0 0 0" xyz="-3.618764437576268e-18 0.010000000000000009 -6.938893903907228e-18"/>
-    <mass value="0.03652101459798134"/>
-    <inertia ixx="7e-06" ixy="0.0" ixz="-0.0" iyy="1.1e-05" iyz="0.0" izz="7e-06"/>
+    <origin rpy="0 0 0" xyz="6.938893903907228e-18 0.009000000000000001 1.3877787807814457e-17"/>
+    <mass value="0.1"/>
+    <inertia ixx="3.239e-05" ixy="0.0" ixz="0.0" iyy="6e-06" iyz="0.0" izz="2.3e-06"/>
   </inertial>
   <visual>
-    <origin rpy="0 0 0" xyz="-0.0 -0.07239 -0.025"/>
+    <geometry>
+      <cylinder length="0.018" radius="0.0215"/>
+    </geometry>
+    <material name="black">
+      <color rgba="0 0 0 1"/>
+    </material>
+  </visual>
+  <collision>
+    <geometry>
+      <cylinder length="0.018" radius="0.0215"/>
+    </geometry>
+  </collision>
+  <!-- <visual>
+    <origin rpy="0 0 0" xyz="-0.025 -0.053 -0.0215"/>
     <geometry>
       <mesh filename="package://bot_description/meshes/wheel_2_1.stl" scale="0.001 0.001 0.001"/>
@@ -38,41 +71,25 @@
   </visual>
   <collision>
-    <origin rpy="0 0 0" xyz="-0.0 -0.07239 -0.025"/>
+    <origin rpy="0 0 0" xyz="-0.025 -0.053 -0.0215"/>
     <geometry>
       <mesh filename="package://bot_description/meshes/wheel_2_1.stl" scale="0.001 0.001 0.001"/>
     </geometry>
-  </collision>
-</link>
-<link name="wheel_1_1">
-  <inertial>
-    <origin rpy="0 0 0" xyz="-3.618764437576268e-18 -0.010000000000000009 -6.938893903907228e-18"/>
-    <mass value="0.03652101459798134"/>
-    <inertia ixx="7e-06" ixy="-0.0" ixz="-0.0" iyy="1.1e-05" iyz="0.0" izz="7e-06"/>
-  </inertial>
-  <visual>
-    <origin rpy="0 0 0" xyz="-0.0 0.07239 -0.025"/>
-    <geometry>
-      <mesh filename="package://bot_description/meshes/wheel_1_1.stl" scale="0.001 0.001 0.001"/>
-    </geometry>
-    <material name="silver"/>
-  </visual>
-  <collision>
-    <origin rpy="0 0 0" xyz="-0.0 0.07239 -0.025"/>
-    <geometry>
-      <mesh filename="package://bot_description/meshes/wheel_1_1.stl" scale="0.001 0.001 0.001"/>
-    </geometry>
-  </collision>
+  </collision> -->
 </link>
 <joint name="Rev1" type="continuous">
-  <origin rpy="0 0 0" xyz="0.0 0.07239 0.025"/>
+  <origin rpy="-1.5708 0 0" xyz="0.025 -0.06 0.0215"/>
+  <parent link="base_link"/>
+  <child link="wheel_1_1"/>
+  <axis xyz="0.0 0.0 1.0"/>
+  <limit effort="10000" velocity="1000"/>
+  <joint_properties damping="1.0" friction="1.0"/>
+</joint>
+<joint name="Rev2" type="continuous">
+  <origin rpy="-1.5708 0 0" xyz="0.025 0.06 0.0215"/>
   <parent link="base_link"/>
   <child link="wheel_2_1"/>
-  <axis xyz="0.0 1.0 0.0"/>
-</joint>
-<joint name="Rev2" type="continuous">
-  <origin rpy="0 0 0" xyz="0.0 -0.07239 0.025"/>
-  <parent link="base_link"/>
-  <child link="wheel_1_1"/>
-  <axis xyz="0.0 -1.0 0.0"/>
+  <axis xyz="0.0 0.0 1.0"/>
+  <limit effort="10000" velocity="1000"/>
+  <joint_properties damping="1.0" friction="1.0"/>
 </joint>
 </robot>

Commit message: changed urdf orgin for pid

File: src/bot_description/urdf/bot.xacro (robot description, xacro)
@@ -26,9 +26,10 @@
 <link name="wheel_1_1">
   <inertial>
-    <origin rpy="0 0 0" xyz="3.469446951953614e-18 -0.009000000000000001 1.0408340855860843e-17"/>
-    <mass value="0.0243098481570003"/>
-    <inertia ixx="3e-06" ixy="0.0" ixz="0.0" iyy="6e-06" iyz="-0.0" izz="3e-06"/>
+    <mass value="0.5"/>
+    <inertia ixx="0.00014299291666666666" ixy="0" ixz="0" iyy="0.00014299291666666666" iyz="0" izz="0.0002739025"/>
+    <origin rpy="0.0 0.0 0.0" xyz="0.0 0.0 0.0"/>
   </inertial>
   <visual>
+    <origin rpy="-1.5708 0 0" xyz="0.025 -0.06 0.0215"/>
     <geometry>
       <cylinder length="0.018" radius="0.0215"/>
@@ -46,9 +47,10 @@
 <link name="wheel_2_1">
   <inertial>
-    <origin rpy="0 0 0" xyz="6.938893903907228e-18 0.009000000000000001 1.3877787807814457e-17"/>
-    <mass value="0.1"/>
-    <inertia ixx="3.239e-05" ixy="0.0" ixz="0.0" iyy="6e-06" iyz="0.0" izz="2.3e-06"/>
+    <mass value="0.5"/>
+    <inertia ixx="0.00014299291666666666" ixy="0" ixz="0" iyy="0.00014299291666666666" iyz="0" izz="0.0002739025"/>
+    <origin rpy="0.0 0.0 0.0" xyz="0.0 0.0 0.0"/>
   </inertial>
   <visual>
+    <origin rpy="-1.5708 0 0" xyz="0.025 0.06 0.0215"/>
     <geometry>
       <cylinder length="0.018" radius="0.0215"/>
@@ -78,5 +80,4 @@
 </link>
 <joint name="Rev1" type="continuous">
-  <origin rpy="-1.5708 0 0" xyz="0.025 -0.06 0.0215"/>
   <parent link="base_link"/>
   <child link="wheel_1_1"/>
@@ -86,5 +87,4 @@
 </joint>
 <joint name="Rev2" type="continuous">
-  <origin rpy="-1.5708 0 0" xyz="0.025 0.06 0.0215"/>
   <parent link="base_link"/>
   <child link="wheel_2_1"/>

Commit message: changed orgin values

File: src/bot_description/urdf/bot.xacro (robot description, xacro)
@@ -1,95 +1,86 @@
-<?xml version="1.0" ?>
+<?xml version="1.0"?>
 <robot name="bot" xmlns:xacro="http://www.ros.org/wiki/xacro">
-<xacro:include filename="$(find bot_description)/urdf/materials.xacro" />
-<xacro:include filename="$(find bot_description)/urdf/bot.trans" />
-<xacro:include filename="$(find bot_description)/urdf/bot.gazebo" />
-<link name="base_link">
-  <inertial>
-    <origin rpy="0 0 0" xyz="-0.0009636587923201293 1.0904768733166021e-17 0.021032044779261124"/>
-    <mass value="0.11050949445484062"/>
-    <inertia ixx="9e-05" ixy="-0.0" ixz="-1e-06" iyy="9.3e-05" iyz="0.0" izz="0.00018"/>
-  </inertial>
-  <visual>
-    <origin rpy="0 0 0" xyz="0 0 0"/>
-    <geometry>
-      <mesh filename="package://bot_description/meshes/base_link.stl" scale="0.001 0.001 0.001"/>
-    </geometry>
-    <material name="silver"/>
-  </visual>
-  <collision>
-    <origin rpy="0 0 0" xyz="0 0 0"/>
-    <geometry>
-      <mesh filename="package://bot_description/meshes/base_link.stl" scale="0.001 0.001 0.001"/>
-    </geometry>
-  </collision>
-</link>
-<link name="wheel_1_1">
-  <inertial>
-    <mass value="0.5"/>
-    <inertia ixx="0.00014299291666666666" ixy="0" ixz="0" iyy="0.00014299291666666666" iyz="0" izz="0.0002739025"/>
-    <origin rpy="0.0 0.0 0.0" xyz="0.0 0.0 0.0"/>
-  </inertial>
-  <visual>
-    <origin rpy="-1.5708 0 0" xyz="0.025 -0.06 0.0215"/>
-    <geometry>
-      <cylinder length="0.018" radius="0.0215"/>
-    </geometry>
-    <material name="black">
-      <color rgba="0 0 0 1"/>
-    </material>
-  </visual>
-  <collision>
-    <geometry>
-      <cylinder length="0.018" radius="0.0215"/>
-    </geometry>
-  </collision>
-</link>
-<link name="wheel_2_1">
-  <inertial>
-    <mass value="0.5"/>
-    <inertia ixx="0.00014299291666666666" ixy="0" ixz="0" iyy="0.00014299291666666666" iyz="0" izz="0.0002739025"/>
-    <origin rpy="0.0 0.0 0.0" xyz="0.0 0.0 0.0"/>
-  </inertial>
-  <visual>
-    <origin rpy="-1.5708 0 0" xyz="0.025 0.06 0.0215"/>
-    <geometry>
-      <cylinder length="0.018" radius="0.0215"/>
-    </geometry>
-    <material name="black">
-      <color rgba="0 0 0 1"/>
-    </material>
-  </visual>
-  <collision>
-    <geometry>
-      <cylinder length="0.018" radius="0.0215"/>
-    </geometry>
-  </collision>
-  <!-- <visual>
-    <origin rpy="0 0 0" xyz="-0.025 -0.053 -0.0215"/>
-    <geometry>
-      <mesh filename="package://bot_description/meshes/wheel_2_1.stl" scale="0.001 0.001 0.001"/>
-    </geometry>
-    <material name="silver"/>
-  </visual>
-  <collision>
-    <origin rpy="0 0 0" xyz="-0.025 -0.053 -0.0215"/>
-    <geometry>
-      <mesh filename="package://bot_description/meshes/wheel_2_1.stl" scale="0.001 0.001 0.001"/>
-    </geometry>
-  </collision> -->
-</link>
-<joint name="Rev1" type="continuous">
-  <parent link="base_link"/>
-  <child link="wheel_1_1"/>
-  <axis xyz="0.0 0.0 1.0"/>
-  <limit effort="10000" velocity="1000"/>
-  <joint_properties damping="1.0" friction="1.0"/>
-</joint>
-<joint name="Rev2" type="continuous">
-  <parent link="base_link"/>
-  <child link="wheel_2_1"/>
-  <axis xyz="0.0 0.0 1.0"/>
-  <limit effort="10000" velocity="1000"/>
-  <joint_properties damping="1.0" friction="1.0"/>
-</joint>
+  <xacro:include filename="$(find bot_description)/urdf/materials.xacro" />
+  <xacro:include filename="$(find bot_description)/urdf/bot.trans" />
+  <xacro:include filename="$(find bot_description)/urdf/bot.gazebo" />
+  <link name="base_link">
+    <inertial>
+      <origin rpy="0 0 0" xyz="-0.0009636587923201293 1.0904768733166021e-17 0.021032044779261124" />
+      <mass value="0.11050949445484062" />
+      <inertia ixx="9e-05" ixy="-0.0" ixz="-1e-06" iyy="9.3e-05" iyz="0.0" izz="0.00018" />
+    </inertial>
+    <visual>
+      <origin rpy="0 0 0" xyz="0 0 0" />
+      <geometry>
+        <mesh filename="package://bot_description/meshes/base_link.stl" scale="0.001 0.001 0.001" />
+      </geometry>
+      <material name="silver" />
+    </visual>
+    <collision>
+      <origin rpy="0 0 0" xyz="0 0 0" />
+      <geometry>
+        <mesh filename="package://bot_description/meshes/base_link.stl" scale="0.001 0.001 0.001" />
+      </geometry>
+    </collision>
+  </link>
+  <link name="wheel_1_1">
+    <inertial>
+      <origin rpy="-1.5708 0 0" xyz="4.469446951953614e-18 -0.059000000000000001 1.0408340855860843e-17" />
+      <mass value="0.1" />
+      <inertia ixx="0.000014256" ixy="0.0" ixz="0.0" iyy="0.000014256" iyz="-0.0" izz="0.000023113" />
+    </inertial>
+    <visual>
+      <origin rpy="-1.5708 0 0" xyz="0 0 0" />
+      <geometry>
+        <cylinder length="0.018" radius="0.0215" />
+      </geometry>
+      <material name="black">
+        <color rgba="0 0 0 1" />
+      </material>
+    </visual>
+    <collision>
+      <geometry>
+        <cylinder length="0.018" radius="0.0215" />
+      </geometry>
+    </collision>
+  </link>
+  <link name="wheel_2_1">
+    <inertial>
+      <origin rpy="-1.5708 0 0" xyz="6.938893903907228e-18 0.059000000000000001 1.3877787807814457e-17" />
+      <mass value="0.1" />
+      <inertia ixx="0.000014256" ixy="0.0" ixz="0.0" iyy="0.000014256" iyz="-0.0" izz="0.000023113" />
+    </inertial>
+    <visual>
+      <origin rpy="-1.5708 0 0" xyz="0 0 0" />
+      <geometry>
+        <cylinder length="0.018" radius="0.0215" />
+      </geometry>
+      <material name="black">
+        <color rgba="0 0 0 1" />
+      </material>
+    </visual>
+    <collision>
+      <geometry>
+        <cylinder length="0.018" radius="0.0215" />
+      </geometry>
+    </collision>
+  </link>
+<!-- right wheel -->
+  <joint name="Rev1" type="continuous">
+    <parent link="base_link" />
+    <child link="wheel_1_1" />
+    <origin rpy ="0 0 0" xyz= "0.025 -0.06 0.0215"/>
+    <axis xyz="0 1 0"/>
+        <limit effort="10000" velocity="1000" />
+    <joint_properties damping="1.0" friction="1.0" />
+  </joint>
+<!-- leftwheel -->
+  <joint name="Rev2" type="continuous">
+    <parent link="base_link" />
+    <child link="wheel_2_1" />
+    <origin rpy ="0 0 0" xyz= "0.025 0.06 0.0215"/>
+    <axis xyz="0 1 0"/>
+        <limit effort="10000" velocity="1000" />
+    <joint_properties damping="1.0" friction="1.0" />
+  </joint>
 </robot>

Commit message: rectified bot link error due to pid

File: src/bot_description/urdf/bot.xacro (robot description, xacro)
@@ -26,5 +26,5 @@
   <link name="wheel_1_1">
     <inertial>
-      <origin rpy="-1.5708 0 0" xyz="4.469446951953614e-18 -0.059000000000000001 1.0408340855860843e-17" />
+      <origin rpy="-1.5708 0 0" xyz="0 0 0" />
       <mass value="0.1" />
       <inertia ixx="0.000014256" ixy="0.0" ixz="0.0" iyy="0.000014256" iyz="-0.0" izz="0.000023113" />
@@ -40,4 +40,5 @@
     </visual>
     <collision>
+      <origin rpy="-1.5708 0 0" xyz="0 0 0" />
       <geometry>
         <cylinder length="0.018" radius="0.0215" />
@@ -47,5 +48,5 @@
   <link name="wheel_2_1">
     <inertial>
-      <origin rpy="-1.5708 0 0" xyz="6.938893903907228e-18 0.059000000000000001 1.3877787807814457e-17" />
+      <origin rpy="-1.5708 0 0" xyz="0 0 0" />
       <mass value="0.1" />
       <inertia ixx="0.000014256" ixy="0.0" ixz="0.0" iyy="0.000014256" iyz="-0.0" izz="0.000023113" />
@@ -61,4 +62,5 @@
     </visual>
     <collision>
+      <origin rpy="-1.5708 0 0" xyz="0 0 0" />
       <geometry>
         <cylinder length="0.018" radius="0.0215" />
@@ -66,20 +68,20 @@
     </collision>
   </link>
-<!-- right wheel -->
+  <!-- right wheel -->
   <joint name="Rev1" type="continuous">
     <parent link="base_link" />
     <child link="wheel_1_1" />
-    <origin rpy ="0 0 0" xyz= "0.025 -0.06 0.0215"/>
-    <axis xyz="0 1 0"/>
-        <limit effort="10000" velocity="1000" />
+    <origin rpy="0 0 0" xyz="0.025 -0.06 0.0215" />
+    <axis xyz="0 1 0" />
+    <limit effort="10000" velocity="1000" />
     <joint_properties damping="1.0" friction="1.0" />
   </joint>
-<!-- leftwheel -->
+  <!-- leftwheel -->
   <joint name="Rev2" type="continuous">
     <parent link="base_link" />
     <child link="wheel_2_1" />
-    <origin rpy ="0 0 0" xyz= "0.025 0.06 0.0215"/>
-    <axis xyz="0 1 0"/>
-        <limit effort="10000" velocity="1000" />
+    <origin rpy="0 0 0" xyz="0.025 0.06 0.0215" />
+    <axis xyz="0 1 0" />
+    <limit effort="10000" velocity="1000" />
     <joint_properties damping="1.0" friction="1.0" />
   </joint>

Commit message: changed to four wheelbot

File: src/bot_description/urdf/bot.xacro (robot description, xacro)
@@ -68,4 +68,48 @@
     </collision>
   </link>
+  <link name="wheel_1_2">
+    <inertial>
+      <origin rpy="-1.5708 0 0" xyz="0 0 0" />
+      <mass value="0.1" />
+      <inertia ixx="0.000014256" ixy="0.0" ixz="0.0" iyy="0.000014256" iyz="-0.0" izz="0.000023113" />
+    </inertial>
+    <visual>
+      <origin rpy="-1.5708 0 0" xyz="0 0 0" />
+      <geometry>
+        <cylinder length="0.018" radius="0.0215" />
+      </geometry>
+      <material name="black">
+        <color rgba="0 0 0 1" />
+      </material>
+    </visual>
+    <collision>
+      <origin rpy="-1.5708 0 0" xyz="0 0 0" />
+      <geometry>
+        <cylinder length="0.018" radius="0.0215" />
+      </geometry>
+    </collision>
+  </link>
+  <link name="wheel_2_2">
+    <inertial>
+      <origin rpy="-1.5708 0 0" xyz="0 0 0" />
+      <mass value="0.1" />
+      <inertia ixx="0.000014256" ixy="0.0" ixz="0.0" iyy="0.000014256" iyz="-0.0" izz="0.000023113" />
+    </inertial>
+    <visual>
+      <origin rpy="-1.5708 0 0" xyz="0 0 0" />
+      <geometry>
+        <cylinder length="0.018" radius="0.0215" />
+      </geometry>
+      <material name="black">
+        <color rgba="0 0 0 1" />
+      </material>
+    </visual>
+    <collision>
+      <origin rpy="-1.5708 0 0" xyz="0 0 0" />
+      <geometry>
+        <cylinder length="0.018" radius="0.0215" />
+      </geometry>
+    </collision>
+  </link>
   <!-- right wheel -->
   <joint name="Rev1" type="continuous">
@@ -73,4 +117,12 @@
     <child link="wheel_1_1" />
     <origin rpy="0 0 0" xyz="0.025 -0.06 0.0215" />
+    <axis xyz="0 1 0" />
+    <limit effort="10000" velocity="1000" />
+    <joint_properties damping="1.0" friction="1.0" />
+  </joint>
+  <joint name="Rev3" type="continuous">
+    <parent link="base_link" />
+    <child link="wheel_1_2" />
+    <origin rpy="0 0 0" xyz="-0.025 0.06 0.0215" />
     <axis xyz="0 1 0" />
     <limit effort="10000" velocity="1000" />
@@ -86,3 +138,11 @@
     <joint_properties damping="1.0" friction="1.0" />
   </joint>
+  <joint name="Rev4" type="continuous">
+    <parent link="base_link" />
+    <child link="wheel_2_2" />
+    <origin rpy="0 0 0" xyz="-0.025 -0.06 0.0215" />
+    <axis xyz="0 1 0" />
+    <limit effort="10000" velocity="1000" />
+    <joint_properties damping="1.0" friction="1.0" />
+  </joint>
 </robot>

Commit message: changed sane names for joints and links

File: src/bot_description/urdf/bot.xacro (robot description, xacro)
@@ -24,5 +24,5 @@
     </collision>
   </link>
-  <link name="wheel_1_1">
+  <link name="front_wheel_right_link">
     <inertial>
       <origin rpy="-1.5708 0 0" xyz="0 0 0" />
@@ -46,5 +46,5 @@
     </collision>
   </link>
-  <link name="wheel_2_1">
+  <link name="front_wheel_left_link">
     <inertial>
       <origin rpy="-1.5708 0 0" xyz="0 0 0" />
@@ -68,5 +68,5 @@
     </collision>
   </link>
-  <link name="wheel_1_2">
+  <link name="rear_wheel_right_link">
     <inertial>
       <origin rpy="-1.5708 0 0" xyz="0 0 0" />
@@ -90,5 +90,5 @@
     </collision>
   </link>
-  <link name="wheel_2_2">
+  <link name="rear_wheel_left_link">
     <inertial>
       <origin rpy="-1.5708 0 0" xyz="0 0 0" />
@@ -113,7 +113,32 @@
   </link>
   <!-- right wheel -->
-  <joint name="Rev1" type="continuous">
+  <joint name="front_right_joint" type="continuous">
     <parent link="base_link" />
-    <child link="wheel_1_1" />
+    <child link="front_wheel_right_link" />
+    <origin rpy="0 0 0" xyz="-0.025 0.06 0.0215" />
+    <axis xyz="0 1 0" />
+    <limit effort="10000" velocity="1000" />
+    <joint_properties damping="1.0" friction="1.0" />
+  </joint>
+  <joint name="front_left_joint" type="continuous">
+    <parent link="base_link" />
+    <child link="front_wheel_left_link" />
+    <origin rpy="0 0 0" xyz="-0.025 -0.06 0.0215" />
+    <axis xyz="0 1 0" />
+    <limit effort="10000" velocity="1000" />
+    <joint_properties damping="1.0" friction="1.0" />
+  </joint>
+  <!-- leftwheel -->
+  <joint name="rear_right_joint" type="continuous">
+    <parent link="base_link" />
+    <child link="rear_wheel_right_link" />
+    <origin rpy="0 0 0" xyz="0.025 0.06 0.0215" />
+    <axis xyz="0 1 0" />
+    <limit effort="10000" velocity="1000" />
+    <joint_properties damping="1.0" friction="1.0" />
+  </joint>
+  <joint name="rear_left_joint" type="continuous">
+    <parent link="base_link" />
+    <child link="rear_wheel_left_link" />
     <origin rpy="0 0 0" xyz="0.025 -0.06 0.0215" />
     <axis xyz="0 1 0" />
@@ -121,28 +146,3 @@
     <joint_properties damping="1.0" friction="1.0" />
   </joint>
-  <joint name="Rev3" type="continuous">
-    <parent link="base_link" />
-    <child link="wheel_1_2" />
-    <origin rpy="0 0 0" xyz="-0.025 0.06 0.0215" />
-    <axis xyz="0 1 0" />
-    <limit effort="10000" velocity="1000" />
-    <joint_properties damping="1.0" friction="1.0" />
-  </joint>
-  <!-- leftwheel -->
-  <joint name="Rev2" type="continuous">
-    <parent link="base_link" />
-    <child link="wheel_2_1" />
-    <origin rpy="0 0 0" xyz="0.025 0.06 0.0215" />
-    <axis xyz="0 1 0" />
-    <limit effort="10000" velocity="1000" />
-    <joint_properties damping="1.0" friction="1.0" />
-  </joint>
-  <joint name="Rev4" type="continuous">
-    <parent link="base_link" />
-    <child link="wheel_2_2" />
-    <origin rpy="0 0 0" xyz="-0.025 -0.06 0.0215" />
-    <axis xyz="0 1 0" />
-    <limit effort="10000" velocity="1000" />
-    <joint_properties damping="1.0" friction="1.0" />
-  </joint>
 </robot>

Commit message: changed acceleration,finalised

File: src/bot_description/urdf/bot.xacro (robot description, xacro)
@@ -6,19 +6,19 @@
 <link name="base_link">
 <inertial>
-<origin rpy="0 0 0" xyz="-0.0009636587923201293 1.0904768733166021e-17 0.021032044779261124" />
+<origin rpy="0 0 0" xyz="0 0 0" />
 <mass value="0.11050949445484062" />
 <inertia ixx="9e-05" ixy="-0.0" ixz="-1e-06" iyy="9.3e-05" iyz="0.0" izz="0.00018" />
 </inertial>
 <visual>
-<origin rpy="0 0 0" xyz="0 0 0" />
+<origin rpy="0 0 0" xyz="-0.081 -0.0793 -0.043" />
 <geometry>
-<mesh filename="package://bot_description/meshes/base_link.stl" scale="0.001 0.001 0.001" />
+<mesh filename="package://bot_description/meshes/base.stl" scale="0.001 0.001 0.001" />
 </geometry>
 <material name="silver" />
 </visual>
 <collision>
-<origin rpy="0 0 0" xyz="0 0 0" />
+<origin rpy="0 0 0" xyz="-0.08 -0.0793 -0.043" />
 <geometry>
-<mesh filename="package://bot_description/meshes/base_link.stl" scale="0.001 0.001 0.001" />
+<mesh filename="package://bot_description/meshes/base.stl" scale="0.001 0.001 0.001" />
 </geometry>
 </collision>
@@ -116,5 +116,5 @@
 <parent link="base_link" />
 <child link="front_wheel_right_link" />
-<origin rpy="0 0 0" xyz="-0.025 0.06 0.0215" />
+<origin rpy="0 0 0" xyz="-0.028 0.06 0.0215" />
 <axis xyz="0 1 0" />
 <limit effort="10000" velocity="1000" />
@@ -124,5 +124,5 @@
 <parent link="base_link" />
 <child link="front_wheel_left_link" />
-<origin rpy="0 0 0" xyz="-0.025 -0.06 0.0215" />
+<origin rpy="0 0 0" xyz="-0.029 -0.06 0.0215" />
 <axis xyz="0 1 0" />
 <limit effort="10000" velocity="1000" />
@@ -133,5 +133,5 @@
 <parent link="base_link" />
 <child link="rear_wheel_right_link" />
-<origin rpy="0 0 0" xyz="0.025 0.06 0.0215" />
+<origin rpy="0 0 0" xyz="0.028 0.06 0.0215" />
 <axis xyz="0 1 0" />
 <limit effort="10000" velocity="1000" />
@@ -141,5 +141,5 @@
 <parent link="base_link" />
 <child link="rear_wheel_left_link" />
-<origin rpy="0 0 0" xyz="0.025 -0.06 0.0215" />
+<origin rpy="0 0 0" xyz="0.029 -0.06 0.0215" />
 <axis xyz="0 1 0" />
 <limit effort="10000" velocity="1000" />
