Commit message: rebased to old description and changed gazebo parameters

File: src/flipbot2_description/urdf/bot.xacro (robot description, xacro)
@@ -34,7 +34,7 @@
         </visual>
         <collision>
-            <origin rpy="0 0 0" xyz="0 0 0 " />
-            <geometry>
-                <box size="0.6 0.1 0.2"/>
+            <origin rpy="0 0 0" xyz="0 0 0.02 " />
+            <geometry>
+                <box size="0.13 0.13 0.005"/>
                 <!-- <mesh filename="package://flipbot_description/meshes/base.stl" scale="0.001 0.001 0.001" /> -->
             </geometry>
@@ -128,5 +128,5 @@
             <origin rpy="-1.5708 0 0" xyz="0 0 0" />
             <geometry>
-                <cylinder length="0.018" radius="0.0215" />
+                <cylinder length="0.005" radius="0.01" />
             </geometry>
         </collision>
@@ -150,5 +150,5 @@
             <origin rpy="-1.5708 0 0" xyz="0 0 0" />
             <geometry>
-                <cylinder length="0.018" radius="0.0215" />
+                <cylinder length="0.005" radius="0.01" />
             </geometry>
         </collision>

Commit message: gazebo launch

File: src/flipbot2_description/urdf/bot.xacro (robot description, xacro)
@@ -41,5 +41,5 @@
         </collision>
     </link>
-    <link name="aruco_tag">
+    <!-- <link name="aruco_tag">
         <visual>
             <origin rpy="0 0 0" xyz="0 0 0.12" />
@@ -65,5 +65,5 @@
             </xacro:if>
         </visual>
-    </link>
+    </link> -->
     <link name="rear_wheel_right_link">
         <inertial>
@@ -160,9 +160,9 @@
     </joint>
     <!-- aruco tags -->
-    <joint name="aruco_joint" type="fixed">
+    <!-- <joint name="aruco_joint" type="fixed">
         <parent link="base_link" />
         <child link="aruco_tag" />
         <origin rpy="0 0 0" xyz="0 0 0" />
-    </joint>
+    </joint> -->
     <!-- leftwheel -->
     <joint name="right_joint" type="continuous">

Commit message: teleop working for flipbot2

File: src/flipbot2_description/urdf/bot.xacro (robot description, xacro)
@@ -5,4 +5,5 @@
     <xacro:include filename="$(find flipbot2_description)/urdf/bot.trans" />
     <xacro:include filename="$(find flipbot2_description)/urdf/bot.gazebo" />
+    <xacro:include filename="$(find flipbot2_description)/urdf/inertia.xacro" />
     <xacro:arg name="index" default='1' />
     <xacro:arg name="index_1" default='False' />
@@ -10,12 +11,4 @@
     <xacro:arg name="index_3" default='False' />
     <xacro:arg name="index_4" default='False' />
-    <xacro:property name="castor_mount_link_length_width_height" value="0.1145 0.10 0.0057" />
-    <xacro:property name="castor_mount_link_length" value="0.1145" />
-    <xacro:property name="castor_mount_link_width" value="0.10" />
-    <xacro:property name="castor_mount_link_height" value="0.0057" />
-    <xacro:property name="castor_mount_link_mass" value="0.25"/> <!--0.25 kg-->
-    <xacro:property name="castor_wheel_length" value="0.049" />
-    <xacro:property name="castor_wheel_radius" value="0.07925" />
-    <xacro:property name="castor_wheel_mass" value="2"/> <!--2 kg-->
     <link name="dummy">
     </link>
@@ -41,5 +34,5 @@
         </collision>
     </link>
-    <!-- <link name="aruco_tag">
+    <link name="aruco_tag">
         <visual>
             <origin rpy="0 0 0" xyz="0 0 0.12" />
@@ -65,11 +58,12 @@
             </xacro:if>
         </visual>
-    </link> -->
+    </link>
     <link name="rear_wheel_right_link">
-        <inertial>
-            <origin rpy="-1.5708 0 0" xyz="0 0 0" />
-            <mass value="0.1" />
-            <inertia ixx="0.000014256" ixy="0.0" ixz="0.0" iyy="0.000014256" iyz="-0.0" izz="0.000023113" />
-        </inertial>
+      <xacro:cylinder_inertia m="0.1"
+                              r="0.0215"
+                              l="0.018"
+                              o_xyz="0.0 0.0 0.0"
+                              o_rpy="${pi/2.0} 0.0 0.0" >
+      </xacro:cylinder_inertia>
         <visual>
             <origin rpy="-1.5708 0 0" xyz="0 0 0" />
@@ -89,9 +83,10 @@
     </link>
     <link name="rear_wheel_left_link">
-        <inertial>
-            <origin rpy="-1.5708 0 0" xyz="0 0 0" />
-            <mass value="0.1" />
-            <inertia ixx="0.000014256" ixy="0.0" ixz="0.0" iyy="0.000014256" iyz="-0.0" izz="0.000023113" />
-        </inertial>
+      <xacro:cylinder_inertia m="0.1"
+                              r="0.0215"
+                              l="0.018"
+                              o_xyz="0.0 0.0 0.0"
+                              o_rpy="${pi/2.0} 0.0 0.0" >
+      </xacro:cylinder_inertia>
         <visual>
             <origin rpy="-1.5708 0 0" xyz="0 0 0" />
@@ -119,5 +114,5 @@
             <origin rpy="-1.5708 0 0" xyz="0 0 0" />
             <geometry>
-                <cylinder length="0.005" radius="0.01" />
+                <cylinder length="0.005" radius="0.008" />
             </geometry>
             <material name="black">
@@ -128,5 +123,5 @@
             <origin rpy="-1.5708 0 0" xyz="0 0 0" />
             <geometry>
-                <cylinder length="0.005" radius="0.01" />
+                <cylinder length="0.005" radius="0.008" />
             </geometry>
         </collision>
@@ -141,5 +136,5 @@
             <origin rpy="-1.5708 0 0" xyz="0 0 0" />
             <geometry>
-                <cylinder length="0.005" radius="0.01" />
+                <cylinder length="0.005" radius="0.008" />
             </geometry>
             <material name="black">
@@ -150,5 +145,5 @@
             <origin rpy="-1.5708 0 0" xyz="0 0 0" />
             <geometry>
-                <cylinder length="0.005" radius="0.01" />
+                <cylinder length="0.005" radius="0.008" />
             </geometry>
         </collision>

Commit message: uncommented aruco joints

File: src/flipbot2_description/urdf/bot.xacro (robot description, xacro)
@@ -155,9 +155,9 @@
     </joint>
     <!-- aruco tags -->
-    <!-- <joint name="aruco_joint" type="fixed">
+     <joint name="aruco_joint" type="fixed">
         <parent link="base_link" />
         <child link="aruco_tag" />
         <origin rpy="0 0 0" xyz="0 0 0" />
-    </joint> -->
+    </joint>
     <!-- leftwheel -->
     <joint name="right_joint" type="continuous">
